Commit message: Restructure envs, add baselines

File: siamrl/envs/data/plane.urdf (robot description, URDF)
Before this commit: robot plane, 1 links, 0 joints
Links:
- link planeLink: geometry collision box size=0.625 0.625 0.1; visual box size=0.625 0.625 0.1

Commit message: Fix QNetwork. Add DQN example

File: siamrl/envs/data/plane.urdf (robot description, URDF)
Before this commit: robot plane, 1 links, 0 joints
Links:
- link planeLink: geometry collision box size=0.4375 0.5625 0.1; visual box size=0.4375 0.5625 0.1

Commit message: Add rewards

File: siamrl/envs/data/plane.urdf (robot description, URDF)
Before this commit: robot plane, 1 links, 0 joints
Links:
- link planeLink: geometry collision box size=0.4375 0.5625 0.1; visual box size=0.4375 0.5625 0.0999

Commit message: Add train utils

File: siamrl/envs/data/plane.urdf (robot description, URDF)
Before this commit: robot plane, 1 links, 0 joints
Links:
- link planeLink: geometry collision box size=10.4375 10.5625 0.1; visual box size=10.4375 10.5625 0.0999

Commit message: Add goal to stack envs

File: siamrl/envs/data/plane.urdf (robot description, URDF)
Before this commit: robot plane, 1 links, 0 joints
Links:
- link planeLink: geometry collision box size=1. 1. 0.2; visual box size=1. 1. .1999
