Commit message: Change train utils, add network parameters

File: siamrl/envs/data/generated/b000.urdf (robot description, URDF)
Before this commit: robot b000, 1 links, 0 joints
Links:
- link link: mass 0.910073532103378 -> 0.3803333610454284

File: siamrl/envs/data/generated/b001.urdf (robot description, URDF)
Before this commit: robot b001, 1 links, 0 joints
Links:
- link link: mass 0.936104906496196 -> 1.0435000257485822

File: siamrl/envs/data/generated/b002.urdf (robot description, URDF)
Before this commit: robot b002, 1 links, 0 joints
Links:
- link link: mass 1.2187507352823632 -> 0.6518184963505628

File: siamrl/envs/data/generated/b003.urdf (robot description, URDF)
Before this commit: robot b003, 1 links, 0 joints
Links:
- link link: mass 0.5514613687047697 -> 0.6325435269830988

File: siamrl/envs/data/generated/b004.urdf (robot description, URDF)
Before this commit: robot b004, 1 links, 0 joints
Links:
- link link: mass 0.7503186961495705 -> 0.488818153096632

File: siamrl/envs/data/generated/b005.urdf (robot description, URDF)
Before this commit: robot b005, 1 links, 0 joints
Links:
- link link: mass 0.8780974940805326 -> 1.031173491633674

File: siamrl/envs/data/generated/b006.urdf (robot description, URDF)
Before this commit: robot b006, 1 links, 0 joints
Links:
- link link: mass 0.7720037968498236 -> 0.6390258933295595

File: siamrl/envs/data/generated/b007.urdf (robot description, URDF)
Before this commit: robot b007, 1 links, 0 joints
Links:
- link link: mass 0.4623162628541564 -> 0.8637245303969006

File: siamrl/envs/data/generated/b008.urdf (robot description, URDF)
Before this commit: robot b008, 1 links, 0 joints
Links:
- link link: mass 0.9900839543435379 -> 0.5199632323270686

File: siamrl/envs/data/generated/b009.urdf (robot description, URDF)
Before this commit: robot b009, 1 links, 0 joints
Links:
- link link: mass 0.6133836526175885 -> 0.44140321453851034

File: siamrl/envs/data/generated/b010.urdf (robot description, URDF)
Before this commit: robot b010, 1 links, 0 joints
Links:
- link link: mass 0.4969842955309114 -> 0.5892503749161789

File: siamrl/envs/data/generated/b011.urdf (robot description, URDF)
Before this commit: robot b011, 1 links, 0 joints
Links:
- link link: mass 0.708592670511894 -> 0.8400314024932792

File: siamrl/envs/data/generated/b012.urdf (robot description, URDF)
Before this commit: robot b012, 1 links, 0 joints
Links:
- link link: mass 0.9935073825628783 -> 0.6924523491816446

File: siamrl/envs/data/generated/b013.urdf (robot description, URDF)
Before this commit: robot b013, 1 links, 0 joints
Links:
- link link: mass 0.8109837085024296 -> 0.7741982822285253

File: siamrl/envs/data/generated/b014.urdf (robot description, URDF)
Before this commit: robot b014, 1 links, 0 joints
Links:
- link link: mass 0.6762298336685004 -> 0.6605413109496133

File: siamrl/envs/data/generated/b015.urdf (robot description, URDF)
Before this commit: robot b015, 1 links, 0 joints
Links:
- link link: mass 0.43163948152123327 -> 0.6515867148071639

File: siamrl/envs/data/generated/b016.urdf (robot description, URDF)
Before this commit: robot b016, 1 links, 0 joints
Links:
- link link: mass 1.0103768668135624 -> 0.4054701684626549

File: siamrl/envs/data/generated/b017.urdf (robot description, URDF)
Before this commit: robot b017, 1 links, 0 joints
Links:
- link link: mass 0.8087812641900338 -> 0.9944148872291131

File: siamrl/envs/data/generated/b018.urdf (robot description, URDF)
Before this commit: robot b018, 1 links, 0 joints
Links:
- link link: mass 0.8367950237968973 -> 0.8198544979447115

File: siamrl/envs/data/generated/b019.urdf (robot description, URDF)
Before this commit: robot b019, 1 links, 0 joints
Links:
- link link: mass 0.6523890233526374 -> 0.5758891216291477
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