Commit message: Change object generation process

File: siamrl/envs/data/generated/test000.urdf (robot description, URDF)
Before this commit: robot test000, 1 links, 0 joints
Links:
- link link: mass 0.42798486566239197 -> 0.37431578129087373

File: siamrl/envs/data/generated/test001.urdf (robot description, URDF)
Before this commit: robot test001, 1 links, 0 joints
Links:
- link link: mass 0.2795694386560857 -> 0.36664182416412844

File: siamrl/envs/data/generated/test002.urdf (robot description, URDF)
Before this commit: robot test002, 1 links, 0 joints
Links:
- link link: mass 0.707363738816415 -> 0.3571860748506233

File: siamrl/envs/data/generated/test003.urdf (robot description, URDF)
Before this commit: robot test003, 1 links, 0 joints
Links:
- link link: mass 0.3916961948177337 -> 0.29947077517074927

File: siamrl/envs/data/generated/test004.urdf (robot description, URDF)
Before this commit: robot test004, 1 links, 0 joints
Links:
- link link: mass 0.6212345788832714 -> 0.27685477983353857

File: siamrl/envs/data/generated/test005.urdf (robot description, URDF)
Before this commit: robot test005, 1 links, 0 joints
Links:
- link link: mass 0.5131470829853394 -> 0.33205167870171054

File: siamrl/envs/data/generated/test006.urdf (robot description, URDF)
Before this commit: robot test006, 1 links, 0 joints
Links:
- link link: mass 0.5725563821972616 -> 0.38365633749756634

File: siamrl/envs/data/generated/test007.urdf (robot description, URDF)
Before this commit: robot test007, 1 links, 0 joints
Links:
- link link: mass 0.9662619067182161 -> 0.5464856781827114

File: siamrl/envs/data/generated/test008.urdf (robot description, URDF)
Before this commit: robot test008, 1 links, 0 joints
Links:
- link link: mass 0.363888120454329 -> 0.4183943481398665

File: siamrl/envs/data/generated/test009.urdf (robot description, URDF)
Before this commit: robot test009, 1 links, 0 joints
Links:
- link link: mass 0.3419611906096162 -> 0.38571493826343234

File: siamrl/envs/data/generated/test010.urdf (robot description, URDF)
Before this commit: robot test010, 1 links, 0 joints
Links:
- link link: mass 0.4119306312404156 -> 0.37480419035293755

File: siamrl/envs/data/generated/test011.urdf (robot description, URDF)
Before this commit: robot test011, 1 links, 0 joints
Links:
- link link: mass 0.5946666831933688 -> 0.42320673768616135

File: siamrl/envs/data/generated/test012.urdf (robot description, URDF)
Before this commit: robot test012, 1 links, 0 joints
Links:
- link link: mass 0.8932142138200203 -> 0.2231909871955643

File: siamrl/envs/data/generated/test013.urdf (robot description, URDF)
Before this commit: robot test013, 1 links, 0 joints
Links:
- link link: mass 0.35685258748667975 -> 0.3778682856529963

File: siamrl/envs/data/generated/test014.urdf (robot description, URDF)
Before this commit: robot test014, 1 links, 0 joints
Links:
- link link: mass 0.49520763910168714 -> 0.4568074010299169

File: siamrl/envs/data/generated/test015.urdf (robot description, URDF)
Before this commit: robot test015, 1 links, 0 joints
Links:
- link link: mass 0.5001289140558772 -> 0.43616936285965935

File: siamrl/envs/data/generated/test016.urdf (robot description, URDF)
Before this commit: robot test016, 1 links, 0 joints
Links:
- link link: mass 0.31905604222002015 -> 0.2803088301986506

File: siamrl/envs/data/generated/test017.urdf (robot description, URDF)
Before this commit: robot test017, 1 links, 0 joints
Links:
- link link: mass 0.538309935514701 -> 0.23635556944898026

File: siamrl/envs/data/generated/test018.urdf (robot description, URDF)
Before this commit: robot test018, 1 links, 0 joints
Links:
- link link: mass 0.6095030974777803 -> 0.1996691890966458

File: siamrl/envs/data/generated/test019.urdf (robot description, URDF)
Before this commit: robot test019, 1 links, 0 joints
Links:
- link link: mass 0.6123150378102872 -> 0.3134726049412373
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
Commit message: Change rock generation

File: siamrl/envs/data/generated/test000.urdf (robot description, URDF)
Before this commit: robot test000, 1 links, 0 joints
Links:
- link link: mass 0.37431578129087373 -> 0.42798486566239197

File: siamrl/envs/data/generated/test001.urdf (robot description, URDF)
Before this commit: robot test001, 1 links, 0 joints
Links:
- link link: mass 0.36664182416412844 -> 0.2795694386560857

File: siamrl/envs/data/generated/test002.urdf (robot description, URDF)
Before this commit: robot test002, 1 links, 0 joints
Links:
- link link: mass 0.3571860748506233 -> 0.707363738816415

File: siamrl/envs/data/generated/test003.urdf (robot description, URDF)
Before this commit: robot test003, 1 links, 0 joints
Links:
- link link: mass 0.29947077517074927 -> 0.3916961948177337

File: siamrl/envs/data/generated/test004.urdf (robot description, URDF)
Before this commit: robot test004, 1 links, 0 joints
Links:
- link link: mass 0.27685477983353857 -> 0.6212345788832714

File: siamrl/envs/data/generated/test005.urdf (robot description, URDF)
Before this commit: robot test005, 1 links, 0 joints
Links:
- link link: mass 0.33205167870171054 -> 0.5131470829853394

File: siamrl/envs/data/generated/test006.urdf (robot description, URDF)
Before this commit: robot test006, 1 links, 0 joints
Links:
- link link: mass 0.38365633749756634 -> 0.5725563821972616

File: siamrl/envs/data/generated/test007.urdf (robot description, URDF)
Before this commit: robot test007, 1 links, 0 joints
Links:
- link link: mass 0.5464856781827114 -> 0.9662619067182161

File: siamrl/envs/data/generated/test008.urdf (robot description, URDF)
Before this commit: robot test008, 1 links, 0 joints
Links:
- link link: mass 0.4183943481398665 -> 0.363888120454329

File: siamrl/envs/data/generated/test009.urdf (robot description, URDF)
Before this commit: robot test009, 1 links, 0 joints
Links:
- link link: mass 0.38571493826343234 -> 0.3419611906096162

File: siamrl/envs/data/generated/test010.urdf (robot description, URDF)
Before this commit: robot test010, 1 links, 0 joints
Links:
- link link: mass 0.37480419035293755 -> 0.4119306312404156

File: siamrl/envs/data/generated/test011.urdf (robot description, URDF)
Before this commit: robot test011, 1 links, 0 joints
Links:
- link link: mass 0.42320673768616135 -> 0.5946666831933688

File: siamrl/envs/data/generated/test012.urdf (robot description, URDF)
Before this commit: robot test012, 1 links, 0 joints
Links:
- link link: mass 0.2231909871955643 -> 0.8932142138200203

File: siamrl/envs/data/generated/test013.urdf (robot description, URDF)
Before this commit: robot test013, 1 links, 0 joints
Links:
- link link: mass 0.3778682856529963 -> 0.35685258748667975

File: siamrl/envs/data/generated/test014.urdf (robot description, URDF)
Before this commit: robot test014, 1 links, 0 joints
Links:
- link link: mass 0.4568074010299169 -> 0.49520763910168714

File: siamrl/envs/data/generated/test015.urdf (robot description, URDF)
Before this commit: robot test015, 1 links, 0 joints
Links:
- link link: mass 0.43616936285965935 -> 0.5001289140558772

File: siamrl/envs/data/generated/test016.urdf (robot description, URDF)
Before this commit: robot test016, 1 links, 0 joints
Links:
- link link: mass 0.2803088301986506 -> 0.31905604222002015

File: siamrl/envs/data/generated/test017.urdf (robot description, URDF)
Before this commit: robot test017, 1 links, 0 joints
Links:
- link link: mass 0.23635556944898026 -> 0.538309935514701

File: siamrl/envs/data/generated/test018.urdf (robot description, URDF)
Before this commit: robot test018, 1 links, 0 joints
Links:
- link link: mass 0.1996691890966458 -> 0.6095030974777803

File: siamrl/envs/data/generated/test019.urdf (robot description, URDF)
Before this commit: robot test019, 1 links, 0 joints
Links:
- link link: mass 0.3134726049412373 -> 0.6123150378102872
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