Commit message: Command line applications

File: siamrl/envs/data/generated/10_000.urdf (robot description, URDF)
Before this commit: robot 10_000, 1 links, 0 joints
Links:
- link link: mass 0.16670613952305777 -> 0.4919411929566806

File: siamrl/envs/data/generated/10_001.urdf (robot description, URDF)
Before this commit: robot 10_001, 1 links, 0 joints
Links:
- link link: mass 0.18277434361441808 -> 0.6635095700008632

File: siamrl/envs/data/generated/10_002.urdf (robot description, URDF)
Before this commit: robot 10_002, 1 links, 0 joints
Links:
- link link: mass 0.1708349171940926 -> 0.5562450276593157

File: siamrl/envs/data/generated/10_003.urdf (robot description, URDF)
Before this commit: robot 10_003, 1 links, 0 joints
Links:
- link link: mass 0.18479492382286536 -> 0.576479730355068

File: siamrl/envs/data/generated/10_004.urdf (robot description, URDF)
Before this commit: robot 10_004, 1 links, 0 joints
Links:
- link link: mass 0.17016717264091485 -> 0.43540846350952905

File: siamrl/envs/data/generated/10_005.urdf (robot description, URDF)
Before this commit: robot 10_005, 1 links, 0 joints
Links:
- link link: mass 0.18964436973871956 -> 0.578468337684783

File: siamrl/envs/data/generated/10_006.urdf (robot description, URDF)
Before this commit: robot 10_006, 1 links, 0 joints
Links:
- link link: mass 0.1758882253709621 -> 0.5466387678719461

File: siamrl/envs/data/generated/10_007.urdf (robot description, URDF)
Before this commit: robot 10_007, 1 links, 0 joints
Links:
- link link: mass 0.16173668813935643 -> 0.4851477673501747

File: siamrl/envs/data/generated/10_008.urdf (robot description, URDF)
Before this commit: robot 10_008, 1 links, 0 joints
Links:
- link link: mass 0.19692838532464618 -> 0.42841828155250805

File: siamrl/envs/data/generated/10_009.urdf (robot description, URDF)
Before this commit: robot 10_009, 1 links, 0 joints
Links:
- link link: mass 0.1706143784102041 -> 0.48115334797493137

File: siamrl/envs/data/generated/10_010.urdf (robot description, URDF)
Before this commit: robot 10_010, 1 links, 0 joints
Links:
- link link: mass 0.1736745467614228 -> 0.541253021306179

File: siamrl/envs/data/generated/10_011.urdf (robot description, URDF)
Before this commit: robot 10_011, 1 links, 0 joints
Links:
- link link: mass 0.15706713086586205 -> 0.641728618929903

File: siamrl/envs/data/generated/10_012.urdf (robot description, URDF)
Before this commit: robot 10_012, 1 links, 0 joints
Links:
- link link: mass 0.16483954391417055 -> 0.6529171360502778

File: siamrl/envs/data/generated/10_013.urdf (robot description, URDF)
Before this commit: robot 10_013, 1 links, 0 joints
Links:
- link link: mass 0.16968472154360228 -> 0.4848183472068338

File: siamrl/envs/data/generated/10_014.urdf (robot description, URDF)
Before this commit: robot 10_014, 1 links, 0 joints
Links:
- link link: mass 0.17840542408024987 -> 0.40730946174679344

File: siamrl/envs/data/generated/10_015.urdf (robot description, URDF)
Before this commit: robot 10_015, 1 links, 0 joints
Links:
- link link: mass 0.16031574132284435 -> 0.4148313536935484

File: siamrl/envs/data/generated/10_016.urdf (robot description, URDF)
Before this commit: robot 10_016, 1 links, 0 joints
Links:
- link link: mass 0.1481387875252981 -> 0.6253871378229956

File: siamrl/envs/data/generated/10_017.urdf (robot description, URDF)
Before this commit: robot 10_017, 1 links, 0 joints
Links:
- link link: mass 0.17168899709112806 -> 0.47385385200339997

File: siamrl/envs/data/generated/10_018.urdf (robot description, URDF)
Before this commit: robot 10_018, 1 links, 0 joints
Links:
- link link: mass 0.16147075192863145 -> 0.4552915943334982

File: siamrl/envs/data/generated/10_019.urdf (robot description, URDF)
Before this commit: robot 10_019, 1 links, 0 joints
Links:
- link link: mass 0.16651340718882332 -> 0.49325233208484337
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
Commit message: New objects

File: siamrl/envs/data/generated/10_000.urdf (robot description, URDF)
Before this commit: robot 10_000, 1 links, 0 joints
Links:
- link link: mass 0.4919411929566806 -> 0.4221219827551651

File: siamrl/envs/data/generated/10_001.urdf (robot description, URDF)
Before this commit: robot 10_001, 1 links, 0 joints
Links:
- link link: mass 0.6635095700008632 -> 0.3377752670021354

File: siamrl/envs/data/generated/10_002.urdf (robot description, URDF)
Before this commit: robot 10_002, 1 links, 0 joints
Links:
- link link: mass 0.5562450276593157 -> 0.5515021787458421

File: siamrl/envs/data/generated/10_003.urdf (robot description, URDF)
Before this commit: robot 10_003, 1 links, 0 joints
Links:
- link link: mass 0.576479730355068 -> 0.5129390479376408

File: siamrl/envs/data/generated/10_004.urdf (robot description, URDF)
Before this commit: robot 10_004, 1 links, 0 joints
Links:
- link link: mass 0.43540846350952905 -> 0.5304786878922468

File: siamrl/envs/data/generated/10_005.urdf (robot description, URDF)
Before this commit: robot 10_005, 1 links, 0 joints
Links:
- link link: mass 0.578468337684783 -> 0.3910397192722599

File: siamrl/envs/data/generated/10_006.urdf (robot description, URDF)
Before this commit: robot 10_006, 1 links, 0 joints
Links:
- link link: mass 0.5466387678719461 -> 0.521054560000363

File: siamrl/envs/data/generated/10_007.urdf (robot description, URDF)
Before this commit: robot 10_007, 1 links, 0 joints
Links:
- link link: mass 0.4851477673501747 -> 0.5298926954272123

File: siamrl/envs/data/generated/10_008.urdf (robot description, URDF)
Before this commit: robot 10_008, 1 links, 0 joints
Links:
- link link: mass 0.42841828155250805 -> 0.5086896246990874

File: siamrl/envs/data/generated/10_009.urdf (robot description, URDF)
Before this commit: robot 10_009, 1 links, 0 joints
Links:
- link link: mass 0.48115334797493137 -> 0.4358423305063668

File: siamrl/envs/data/generated/10_010.urdf (robot description, URDF)
Before this commit: robot 10_010, 1 links, 0 joints
Links:
- link link: mass 0.541253021306179 -> 0.5282927266923957

File: siamrl/envs/data/generated/10_011.urdf (robot description, URDF)
Before this commit: robot 10_011, 1 links, 0 joints
Links:
- link link: mass 0.641728618929903 -> 0.4316073889102194

File: siamrl/envs/data/generated/10_012.urdf (robot description, URDF)
Before this commit: robot 10_012, 1 links, 0 joints
Links:
- link link: mass 0.6529171360502778 -> 0.4951342919426195

File: siamrl/envs/data/generated/10_013.urdf (robot description, URDF)
Before this commit: robot 10_013, 1 links, 0 joints
Links:
- link link: mass 0.4848183472068338 -> 0.47889803477740134

File: siamrl/envs/data/generated/10_014.urdf (robot description, URDF)
Before this commit: robot 10_014, 1 links, 0 joints
Links:
- link link: mass 0.40730946174679344 -> 0.5391628121447324

File: siamrl/envs/data/generated/10_015.urdf (robot description, URDF)
Before this commit: robot 10_015, 1 links, 0 joints
Links:
- link link: mass 0.4148313536935484 -> 0.511664122476871

File: siamrl/envs/data/generated/10_016.urdf (robot description, URDF)
Before this commit: robot 10_016, 1 links, 0 joints
Links:
- link link: mass 0.6253871378229956 -> 0.37260419358843055

File: siamrl/envs/data/generated/10_017.urdf (robot description, URDF)
Before this commit: robot 10_017, 1 links, 0 joints
Links:
- link link: mass 0.47385385200339997 -> 0.4364284813352625

File: siamrl/envs/data/generated/10_018.urdf (robot description, URDF)
Before this commit: robot 10_018, 1 links, 0 joints
Links:
- link link: mass 0.4552915943334982 -> 0.44154125776822206

File: siamrl/envs/data/generated/10_019.urdf (robot description, URDF)
Before this commit: robot 10_019, 1 links, 0 joints
Links:
- link link: mass 0.49325233208484337 -> 0.5804344474413985
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