Commit message: New models and changes to baselines

File: siamrl/envs/data/generated/0_0.urdf (robot description, URDF)
Before this commit: robot 0_0, 1 links, 0 joints
Links:
- link link: mass 0.5232968449718013 -> 0.45314713303124377

File: siamrl/envs/data/generated/10_000.urdf (robot description, URDF)
Before this commit: robot 10_000, 1 links, 0 joints
Links:
- link link: mass 0.4221219827551651 -> 0.43011301356661347

File: siamrl/envs/data/generated/10_001.urdf (robot description, URDF)
Before this commit: robot 10_001, 1 links, 0 joints
Links:
- link link: mass 0.3377752670021354 -> 0.5113652302580873

File: siamrl/envs/data/generated/10_002.urdf (robot description, URDF)
Before this commit: robot 10_002, 1 links, 0 joints
Links:
- link link: mass 0.5515021787458421 -> 0.48018499264703957

File: siamrl/envs/data/generated/10_003.urdf (robot description, URDF)
Before this commit: robot 10_003, 1 links, 0 joints
Links:
- link link: mass 0.5129390479376408 -> 0.5908502408839733

File: siamrl/envs/data/generated/10_004.urdf (robot description, URDF)
Before this commit: robot 10_004, 1 links, 0 joints
Links:
- link link: mass 0.5304786878922468 -> 0.497000762769049

File: siamrl/envs/data/generated/10_005.urdf (robot description, URDF)
Before this commit: robot 10_005, 1 links, 0 joints
Links:
- link link: mass 0.3910397192722599 -> 0.47114799807955615

File: siamrl/envs/data/generated/10_006.urdf (robot description, URDF)
Before this commit: robot 10_006, 1 links, 0 joints
Links:
- link link: mass 0.521054560000363 -> 0.3862582377203118

File: siamrl/envs/data/generated/10_007.urdf (robot description, URDF)
Before this commit: robot 10_007, 1 links, 0 joints
Links:
- link link: mass 0.5298926954272123 -> 0.49949666011608757

File: siamrl/envs/data/generated/10_008.urdf (robot description, URDF)
Before this commit: robot 10_008, 1 links, 0 joints
Links:
- link link: mass 0.5086896246990874 -> 0.5488690914718733

File: siamrl/envs/data/generated/10_009.urdf (robot description, URDF)
Before this commit: robot 10_009, 1 links, 0 joints
Links:
- link link: mass 0.4358423305063668 -> 0.5159960250863262

File: siamrl/envs/data/generated/10_010.urdf (robot description, URDF)
Before this commit: robot 10_010, 1 links, 0 joints
Links:
- link link: mass 0.5282927266923957 -> 0.49112918857253146

File: siamrl/envs/data/generated/10_011.urdf (robot description, URDF)
Before this commit: robot 10_011, 1 links, 0 joints
Links:
- link link: mass 0.4316073889102194 -> 0.5748622253568411

File: siamrl/envs/data/generated/10_012.urdf (robot description, URDF)
Before this commit: robot 10_012, 1 links, 0 joints
Links:
- link link: mass 0.4951342919426195 -> 0.598029790190552

File: siamrl/envs/data/generated/10_013.urdf (robot description, URDF)
Before this commit: robot 10_013, 1 links, 0 joints
Links:
- link link: mass 0.47889803477740134 -> 0.5024277599942472

File: siamrl/envs/data/generated/10_014.urdf (robot description, URDF)
Before this commit: robot 10_014, 1 links, 0 joints
Links:
- link link: mass 0.5391628121447324 -> 0.5206426319516478

File: siamrl/envs/data/generated/10_015.urdf (robot description, URDF)
Before this commit: robot 10_015, 1 links, 0 joints
Links:
- link link: mass 0.511664122476871 -> 0.40030189023212337

File: siamrl/envs/data/generated/10_016.urdf (robot description, URDF)
Before this commit: robot 10_016, 1 links, 0 joints
Links:
- link link: mass 0.37260419358843055 -> 0.5350986025822988

File: siamrl/envs/data/generated/10_017.urdf (robot description, URDF)
Before this commit: robot 10_017, 1 links, 0 joints
Links:
- link link: mass 0.4364284813352625 -> 0.7137136667108973

File: siamrl/envs/data/generated/10_018.urdf (robot description, URDF)
Before this commit: robot 10_018, 1 links, 0 joints
Links:
- link link: mass 0.44154125776822206 -> 0.5057580195559434
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
Commit message: Center meshes in oriented bounding box

File: siamrl/envs/data/generated/0_0.urdf (robot description, URDF)
Before this commit: robot 0_0, 1 links, 0 joints
Links:
- link link: mass 0.45314713303124377 -> 0.5324038486184894

File: siamrl/envs/data/generated/0_1.urdf (robot description, URDF)
Before this commit: robot 0_1, 1 links, 0 joints
Links:
- link link: mass 0.5180232589605307 -> 0.46488239672127046

File: siamrl/envs/data/generated/0_2.urdf (robot description, URDF)
Before this commit: robot 0_2, 1 links, 0 joints
Links:
- link link: mass 0.4895828329229362 -> 0.4990635336679104

File: siamrl/envs/data/generated/0_3.urdf (robot description, URDF)
Before this commit: robot 0_3, 1 links, 0 joints
Links:
- link link: mass 0.45911919073260327 -> 0.4757495759273942

File: siamrl/envs/data/generated/0_4.urdf (robot description, URDF)
Before this commit: robot 0_4, 1 links, 0 joints
Links:
- link link: mass 0.5115949791359564 -> 0.4613213503055904

File: siamrl/envs/data/generated/100_000.urdf (robot description, URDF)
Before this commit: robot 100_000, 1 links, 0 joints
Links:
- link link: mass 0.714171532537639 -> 0.4244786576500648

File: siamrl/envs/data/generated/100_001.urdf (robot description, URDF)
Before this commit: robot 100_001, 1 links, 0 joints
Links:
- link link: mass 0.4020695830315688 -> 0.24937097605852238

File: siamrl/envs/data/generated/100_002.urdf (robot description, URDF)
Before this commit: robot 100_002, 1 links, 0 joints
Links:
- link link: mass 0.3718642417863417 -> 0.39092323470156076

File: siamrl/envs/data/generated/100_003.urdf (robot description, URDF)
Before this commit: robot 100_003, 1 links, 0 joints
Links:
- link link: mass 0.2891929184009459 -> 0.32582550019144196

File: siamrl/envs/data/generated/100_004.urdf (robot description, URDF)
Before this commit: robot 100_004, 1 links, 0 joints
Links:
- link link: mass 0.48306255644290486 -> 0.41051363051940915

File: siamrl/envs/data/generated/100_005.urdf (robot description, URDF)
Before this commit: robot 100_005, 1 links, 0 joints
Links:
- link link: mass 0.8162946164300601 -> 0.42190601667307487

File: siamrl/envs/data/generated/100_006.urdf (robot description, URDF)
Before this commit: robot 100_006, 1 links, 0 joints
Links:
- link link: mass 0.6995898261883373 -> 0.514321992250474

File: siamrl/envs/data/generated/100_007.urdf (robot description, URDF)
Before this commit: robot 100_007, 1 links, 0 joints
Links:
- link link: mass 0.29564387462941544 -> 0.390861191882435

File: siamrl/envs/data/generated/100_008.urdf (robot description, URDF)
Before this commit: robot 100_008, 1 links, 0 joints
Links:
- link link: mass 0.18884737392002268 -> 0.3321166952523327

File: siamrl/envs/data/generated/100_009.urdf (robot description, URDF)
Before this commit: robot 100_009, 1 links, 0 joints
Links:
- link link: mass 0.5495065991374553 -> 0.5036505321937563

File: siamrl/envs/data/generated/100_010.urdf (robot description, URDF)
Before this commit: robot 100_010, 1 links, 0 joints
Links:
- link link: mass 0.478385444281879 -> 0.7623521111011357

File: siamrl/envs/data/generated/100_011.urdf (robot description, URDF)
Before this commit: robot 100_011, 1 links, 0 joints
Links:
- link link: mass 0.6759088674757491 -> 0.36766480601314666

File: siamrl/envs/data/generated/100_012.urdf (robot description, URDF)
Before this commit: robot 100_012, 1 links, 0 joints
Links:
- link link: mass 0.6721959382280203 -> 0.3114630755411156

File: siamrl/envs/data/generated/100_013.urdf (robot description, URDF)
Before this commit: robot 100_013, 1 links, 0 joints
Links:
- link link: mass 0.8162168461648424 -> 0.3999969777109329

File: siamrl/envs/data/generated/100_014.urdf (robot description, URDF)
Before this commit: robot 100_014, 1 links, 0 joints
Links:
- link link: mass 0.4741833843884495 -> 0.4716204667607296
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